Commit message: add working 4x4 implementation

File: hoverboard_demo_description/urdf/hoverboard_description.xacro (robot description, xacro)
@@ -37,8 +37,10 @@
         <child link="plate" />
     </joint>
-    <xacro:driving_wheel suffix="left" reflect="1"/>
-    <xacro:driving_wheel suffix="right" reflect="-1"/>
-    <xacro:caster_wheel suffix="front" reflect="1" />
-    <xacro:caster_wheel suffix="back" reflect="-1" />
-    <xacro:hoverboard_ros2_control name="Hoverboard" />
+    <xacro:driving_wheel suffix="front_left" reflect="1" position="0.3"/>
+    <xacro:driving_wheel suffix="front_right" reflect="-1" position="0.3"/>
+    <xacro:driving_wheel suffix="back_left" reflect="1" position="-0.3"/>
+    <xacro:driving_wheel suffix="back_right" reflect="-1" position="-0.3"/>
+    <!-- <xacro:caster_wheel suffix="front" reflect="1" />
+    <xacro:caster_wheel suffix="back" reflect="-1" /> -->
+    <xacro:hoverboard_ros2_control name="hoverboard" />
 </robot>

File: hoverboard_demo_description/urdf/ros2_control.xacro (robot description, xacro)
@@ -2,9 +2,9 @@
 <robot xmlns:xacro="http://www.ros.org/wiki/xacro">
   <xacro:macro name="hoverboard_ros2_control" params="name">
-    <ros2_control name="${name}" type="system">
+    <ros2_control name="${name}_front" type="system">
       <hardware>
         <plugin>hoverboard_hardware_interface/HoverboardHardwareInterface</plugin>
-        <param name="left_wheel_joint_name">driving_wheel_left_joint</param>
-        <param name="right_wheel_joint_name">driving_wheel_right_joint</param>
+        <param name="left_wheel_joint_name">driving_wheel_front_left_joint</param>
+        <param name="right_wheel_joint_name">driving_wheel_front_right_joint</param>
         <param name="loop_rate">50</param>
         <param name="device">/dev/ttyUSB0</param>
@@ -13,10 +13,32 @@
         <param name="encoder_ticks_per_revolution">90</param>
       </hardware>
-      <joint name="driving_wheel_left_joint">
+      <joint name="driving_wheel_front_left_joint">
         <command_interface name="velocity"/>
         <state_interface name="position"/>
         <state_interface name="velocity"/>
       </joint>
-      <joint name="driving_wheel_right_joint">
+      <joint name="driving_wheel_front_right_joint">
+        <command_interface name="velocity"/>
+        <state_interface name="position"/>
+        <state_interface name="velocity"/>
+      </joint>
+    </ros2_control>
+    <ros2_control name="${name}_back" type="system">
+      <hardware>
+        <plugin>hoverboard_hardware_interface/HoverboardHardwareInterface</plugin>
+        <param name="left_wheel_joint_name">driving_wheel_back_left_joint</param>
+        <param name="right_wheel_joint_name">driving_wheel_back_right_joint</param>
+        <param name="loop_rate">50</param>
+        <param name="device">/dev/ttyUSB1</param>
+        <param name="baud_rate">115200</param>
+        <param name="timeout">1000</param>
+        <param name="encoder_ticks_per_revolution">90</param>
+      </hardware>
+      <joint name="driving_wheel_back_left_joint">
+        <command_interface name="velocity"/>
+        <state_interface name="position"/>
+        <state_interface name="velocity"/>
+      </joint>
+      <joint name="driving_wheel_back_right_joint">
         <command_interface name="velocity"/>
         <state_interface name="position"/>

File: hoverboard_demo_description/urdf/wheels.xacro (robot description, xacro)
@@ -2,5 +2,5 @@
 <robot xmlns:xacro="http://ros.org/wiki/xacro">
     <!-- TODO: The model is made in a very simple form, it would be nice to make it a bit better. Is someone willing? -->
-    <xacro:macro name="driving_wheel" params="suffix reflect">
+    <xacro:macro name="driving_wheel" params="suffix reflect position">
         <link name="driving_wheel_${suffix}">
             <visual>
@@ -24,5 +24,5 @@
             <parent link="base_link"/>
             <child link="driving_wheel_${suffix}"/>
-            <origin xyz="0 ${(plate_radius+driving_wheel_thickness+driving_wheel_base_gap-0.195)/2*reflect} 0.038" rpy="0 0 0"/>
+            <origin xyz="${position} ${(plate_radius+driving_wheel_thickness+driving_wheel_base_gap-0.195)/2*reflect} 0.038" rpy="0 0 0"/>
         </joint>
         <gazebo reference="driving_wheel_${suffix}">
